File: vcore-3/eva-loveboard-1.1/PCB/eva-toolboard-20p.kicad_pcb (KiCad board)
At the start: 2 copper layers, 44.1 x 48.8 mm, 16 parts, among them J1 TH0, J10 Neopixel, J2 HEATER, J3 STEPPER, J4 Main connector, J5 HOTENDFAN, J6 PARTFAN_1, J7 PARTFAN_2, J8 ENDSTOP_X, J9 PROBE

Commit message: First draft of the new 2p th board
Parts:
- added J11: ENDSTOP_E, Connector_JST:JST_PH_B2B-PH-K_1x02_P2.00mm_Vertical, B.Cu at (131.8, 101.2)
- J1: footprint Connector_JST:JST_PH_B4B-PH-K_1x04_P2.00mm_Vertical -> Connector_JST:JST_PH_B2B-PH-K_1x02_P2.00mm_Vertical
- TH1: footprint Resistor_THT:R_Axial_DIN0204_L3.6mm_D1.6mm_P7.62mm_Horizontal -> Diode_THT:D_A-405_P7.62mm_Horizontal
- moved J7 1.67 mm to (131.8, 106.2), turned to 0 degrees
- moved J1 1.00 mm to (131.8, 96.2), turned to 0 degrees
Connections:
- J4 pad 1: Net-(J1-Pad4) -> +12V
- J4 pad 2: Net-(J1-Pad3) -> Net-(J4-Pad2)
Routing:
- net Net-(J4-Pad2): track 0.00 -> 21.9 mm
- net Net-(J1-Pad3): track 20.3 -> 0.00 mm
- net Net-(J1-Pad4): track 16.0 -> 0.00 mm
- net +24V: track 70.9 -> 67.0 mm
- net Net-(J4-Pad15): track 48.7 -> 46.7 mm
Other:
- board text added: "Loveboard 1.1"
- board text removed: "Loveboard 1.0"
