File: vcore-3/eva-loveboard-1.1/PCB/eva-toolboard-20p.kicad_sch (KiCad schematic)
At the start: 11 parts, among them J1 TH0, J10 Neopixel, J2 HEATER, J3 STEPPER, J4 Main connector, J5 HOTENDFAN, J6 PARTFAN_1, J7 PARTFAN_2, J8 ENDSTOP_X, J9 PROBE

Commit message: First draft of the new 2p th board
Parts:
- added J11: ENDSTOP_E, Connector_JST:JST_PH_B2B-PH-K_1x02_P2.00mm_Vertical, symbol Connector_Generic:Conn_01x02
- J1: footprint Connector_JST:JST_PH_B4B-PH-K_1x04_P2.00mm_Vertical -> Connector_JST:JST_PH_B2B-PH-K_1x02_P2.00mm_Vertical; symbol Connector_Generic:Conn_01x04 -> Connector_Generic:Conn_01x02
Connections:
- net GND: now also J11.2 (Pin_2)
- net +12V: now reaches J4.1 (Pin_1)
- net +12V: no longer J1.4 (Pin_4)
- net at J4.2 (Pin_2): now also J11.1 (Pin_1); no longer J1.3 (Pin_3)
